Commit message: モデルを修正

File: simple_leg_description/xacro/simple_leg.xacro (robot description, xacro)
@@ -1,5 +1,5 @@
 <?xml version="1.0"?>
-<robot name="MELEW_2L" xmlns:xacro="http://www.ros.org/wiki/xacro">
-    <xacro:include filename="$(find ros_control_tutorial)/xacro/simple_leg_macro.xacro"/>
+<robot name="simple_leg" xmlns:xacro="http://www.ros.org/wiki/xacro">
+    <xacro:include filename="$(find simple_leg_description)/xacro/simple_leg_macro.xacro"/>
     <link name="world"/>
     <xacro:simple_leg_macro parent="world" z_offset="1.0"/>

File: simple_leg_description/xacro/simple_leg_macro.xacro (robot description, xacro)
@@ -25,8 +25,8 @@
         <joint name="base_joint" type="fixed">
             <parent link="${parent}"/>
-            <child link="body_link"/>
+            <child link="base_link"/>
             <origin rpy="0 0 0" xyz="0 0 ${z_offset}"/>
         </joint>
-        <link name="body_link">
+        <link name="base_link">
             <visual>
                 <origin rpy="0 0 0" xyz="0 0 0"/>
@@ -49,9 +49,9 @@
         <!-- Hip_joint & UpperThigh_link -->
         <joint name="Hip" type="revolute">
-            <parent link="body_link"/>
+            <parent link="base_link"/>
             <child link="upperThigh"/>
             <axis xyz="0 1 0"/>
             <origin rpy="0 0 0" xyz="0 0 0.0"/>
-            <limit effort="1000" lower="${radians(-90)}" upper="${radians(90)}" velocity="30.0"/>
+            <limit effort="1000" lower="${radians(-180)}" upper="${radians(180)}" velocity="30.0"/>
         </joint>
         <link name="upperThigh">
@@ -80,5 +80,5 @@
             <axis xyz="0 1 0"/>
             <origin rpy="0 0 0" xyz="0 0 -${l1}"/>
-            <limit effort="1000" lower="${radians(-135)}" upper="${radians(15)}" velocity="30.0"/>
+            <limit effort="1000" lower="${radians(-180)}" upper="${radians(180)}" velocity="30.0"/>
         </joint>
         <link name="lowerThigh">
@@ -124,6 +124,8 @@
         <gazebo>
             <plugin name="gazebo_ros_control" filename="libgazebo_ros_control.so">
-                <robotNamespace>/MELEW_2L</robotNamespace>
+                <!--
                 <robotSimType>gazebo_ros_control/DefaultRobotHWSim</robotSimType>
+                -->
+                <robotSimType>simple_leg_hw_sim/SimpleLegHWSim</robotSimType>
             </plugin>
         </gazebo>
