Commit message: update

File: simple_leg_description/xacro/simple_leg_macro.xacro (robot description, xacro)
@@ -59,5 +59,5 @@
                 <origin rpy="0 0 0" xyz="0 0 -${l1/2}"/>
                 <geometry>
-                    <box size="0.05 0.05 0.2"/>
+                    <box size="0.05 0.05 ${l1}"/>
                 </geometry>
                 <material name="red"/>
@@ -124,7 +124,5 @@
         <gazebo>
             <plugin name="gazebo_ros_control" filename="libgazebo_ros_control.so">
-                <!--
-                <robotSimType>gazebo_ros_control/DefaultRobotHWSim</robotSimType>
-                -->
+                <!--<robotSimType>gazebo_ros_control/DefaultRobotHWSim</robotSimType>-->
                 <robotSimType>simple_leg_hw_sim/SimpleLegHWSim</robotSimType>
             </plugin>
@@ -140,7 +138,4 @@
             <material>Gazebo/Red</material>
         </gazebo>
-        <gazebo reference="Whee_link">
-            <material>Gazebo/White</material>
-        </gazebo>
     </xacro:macro>
 </robot>
